Commit message: sim : update sensor box and livox 3d lidar

File: urdf/gazebo/joint_state_gazebo.xacro (robot description, xacro)
@@ -10,5 +10,4 @@
             <joint_name>wheel_rr_joint</joint_name>
             <joint_name>blade_joint</joint_name>
-            <joint_name>blade_joint</joint_name>
         </plugin>
     </gazebo>

File: urdf/msd700_blade_description.urdf.xacro (robot description, xacro)
@@ -3,11 +3,25 @@
 <!-- ================= INCLUDE ================= -->
     <xacro:include filename="$(find msd700_robot_description)/urdf/commons/msd700_wheel.xacro"/>
-    <xacro:include filename="$(find msd700_robot_description)/urdf/commons/msd700_base.xacro"/>
+    <xacro:include filename="$(find msd700_robot_description)/urdf/commons/msd700_base_only.xacro"/>
+    <xacro:include filename="$(find msd700_robot_description)/urdf/commons/msd700_track.xacro"/>
     <xacro:include filename="$(find msd700_robot_description)/urdf/attachment/msd700_blade.xacro"/>
+    <xacro:include filename="$(find msd700_robot_description)/urdf/sensors/sensor_livox_360.xacro"/>
     <xacro:include filename="$(find msd700_robot_description)/urdf/gazebo/base_control_gazebo.xacro"/>
     <xacro:include filename="$(find msd700_robot_description)/urdf/gazebo/joint_state_gazebo.xacro"/>
+    <xacro:include filename="$(find msd700_robot_description)/urdf/gazebo/sensor_2d_lidar_gazebo.xacro"/>
+    <xacro:include filename="$(find msd700_robot_description)/urdf/gazebo/sensor_imu_gazebo.xacro"/>
+    <xacro:property name="box_weight"       value="0.85" />
+    <xacro:property name="box_width"        value="0.15" />
+    <xacro:property name="box_length"       value="0.3" />
+    <xacro:property name="box_height"       value="0.15" />
+    <xacro:property name="base_width"       value="0.47" />
+    <xacro:property name="base_length"      value="0.866" />
+    <xacro:property name="base_height"      value="0.271" />
 <!-- ================= BASE ================= -->
     <link name="base_footprint"/>
     <xacro:base name="base" parent="base_footprint" xyz="0 0 0.05" rpy="0 0 0"/>
+<!-- ================= TRACK ================= -->
+    <xacro:track name="track_left"  parent="base_link" xyz="-0.285 0.30 0.065" rpy="0 0 0"/>
+    <xacro:track name="track_right" parent="base_link" xyz="-0.285 -0.30 0.065" rpy="0 0 0"/>
 <!-- ================= WHEELS ================= -->
     <xacro:wheel name="wheel_fl" parent="base_link" xyz="0.305 0.30 0.065" rpy="0 0 0"/>
@@ -21,5 +35,5 @@
         <parent link="base_link"/>
         <child link="sensor_box_link"/>
-        <origin xyz="0 0 0.23" rpy="0 0 0"/>
+        <origin xyz="${0.433-(box_length/2)-0.2} ${0.205-(box_width/2)} 0.23" rpy="0 0 0"/>
     </joint>
     <link name="sensor_box_link">
@@ -27,5 +41,5 @@
             <origin xyz="0 0 0.075" rpy="0 0 0"/>
             <geometry>
-                <box size="0.6 0.4 0.15"/>
+                <box size="${box_length} ${box_width} ${box_height}"/>
             </geometry>
             <material name="Gray">
@@ -34,7 +48,7 @@
         </visual>
         <collision>
-            <origin xyz="0 0 0.075" rpy="0 0 0"/>
+            <origin xyz="${0.433-(box_length/2)-0.2} ${0.205-(box_width/2)} 0.075" rpy="0 0 0"/>
             <geometry>
-                <box size="0.6 0.4 0.15"/>
+                <box size="${box_length} ${box_width} ${box_height}"/>
             </geometry>
             <material name="Gray">
@@ -44,10 +58,13 @@
         <inertial>
             <origin xyz="0 0 0.075" rpy="0 0 0"/>
-            <mass value="1.0"/>
+            <mass value="${box_weight}"/>
             <inertia
-                    ixx="${(1/12)*(0.4*0.4 + 0.15*0.15)}"   ixy="0.0" ixz="0.0"
-                    iyy="${(1/12)*(0.6*0.6 + 0.15*0.15)}"   iyz="0.0"
-                    izz="${(1/12)*(0.6*0.6 + 0.4*0.4)}"/>
+                    ixx="${(box_weight/12)*(box_width*box_width + box_height*box_height)}"   ixy="0.0" ixz="0.0"
+                    iyy="${(box_weight/12)*(box_length*box_length + box_height*box_height)}" iyz="0.0"
+                    izz="${(box_weight/12)*(box_length*box_length + box_width*box_width)}"/>
         </inertial>
     </link>
+    <xacro:livox name="livox" parent="sensor_box_link" xyz="-${(box_length/2)-(0.065/2)} -${(box_width/2)-(0.065/2)} ${box_height+0.060/2}" rpy="0 0 0"/>
+    <xacro:lidar_2d_plugin name="livox" topic="/scan"/>
+    <xacro:livox_imu_plugin name="livox"/>
 </robot>
