Commit message: feat : additional 2D lidar plugin and 3D lidar plugin

File: urdf/gazebo/sensor_3d_lidar_gazebo.xacro (robot description, xacro)
@@ -1,25 +1,28 @@
 <?xml version="1.0"?>
 <robot xmlns:xacro="http://ros.org/wiki/xacro">
-  <xacro:macro name="lidar_2d_plugin" params="link_reference topic">
+  <xacro:macro name="lidar_3d_plugin" params="link_reference topic">
     <gazebo reference="${link_reference}">
       <sensor name="${name}" type="gpu_lidar">
         <pose>0 0 0 0 0 0</pose>
+        <topic>${topic}</topic>
+        <gz_frame_id>${link_reference}</gz_frame_id>
         <update_rate>10</update_rate>
+        <always_on>true</always_on>
         <visualize>true</visualize>
-        <topic>${topic}</topic>
-        <ray>
+        <lidar>
           <scan>
             <horizontal>
-              <samples>720</samples>        <!-- resolution -->
+              <!-- 360 degree horizontal -->
+              <samples>360</samples>
               <resolution>1</resolution>
               <min_angle>-3.14159</min_angle>
               <max_angle>3.14159</max_angle>
             </horizontal>
-            <!-- 2D = vertical = 1 -->
             <vertical>
-              <samples>1</samples>
+              <!-- 16 vertical channels, -15 to +15 degrees -->
+              <samples>16</samples>
               <resolution>1</resolution>
-              <min_angle>0</min_angle>
-              <max_angle>0</max_angle>
+              <min_angle>-0.26180</min_angle>  <!-- -15 deg -->
+              <max_angle>0.26180</max_angle>   <!-- +15 deg -->
             </vertical>
           </scan>
@@ -34,5 +37,5 @@
             <stddev>0.01</stddev>
           </noise>
-        </ray>
+        </lidar>
       </sensor>
     </gazebo>

File: urdf/sensors/sensor_livox_360.xacro (robot description, xacro)
@@ -1,4 +1,6 @@
 <?xml version="1.0"?>
 <robot xmlns:xacro="http://ros.org/wiki/xacro">
+    <!-- Include -->
+    <xacro:include filename="$(find msd700_robot_description)/urdf/gazebo/sensor_3d_lidar_gazebo.xacro"/>
     <!-- From MCLA015B spec -->
     <xacro:property name="livox_weight"  value="0.265" />
@@ -43,42 +45,5 @@
             </inertial>
         </link>
-        <gazebo reference="${name}_link">
-            <sensor name="${name}_sensor" type="gpu_lidar">
-                <pose>0 0 0 0 0 0</pose>
-                <topic>/scan</topic>
-                <gz_frame_id>${name}_link</gz_frame_id>
-                <update_rate>10</update_rate>
-                <always_on>true</always_on>
-                <visualize>true</visualize>
-                <lidar>
-                    <scan>
-                        <horizontal>
-                            <!-- 360 degree horizontal -->
-                            <samples>360</samples>
-                            <resolution>1</resolution>
-                            <min_angle>-3.14159</min_angle>
-                            <max_angle>3.14159</max_angle>
-                        </horizontal>
-                        <vertical>
-                            <!-- 16 vertical channels, -15 to +15 degrees -->
-                            <samples>16</samples>
-                            <resolution>1</resolution>
-                            <min_angle>-0.26180</min_angle>  <!-- -15 deg -->
-                            <max_angle>0.26180</max_angle>   <!-- +15 deg -->
-                        </vertical>
-                    </scan>
-                    <range>
-                        <min>0.1</min>
-                        <max>30.0</max>
-                        <resolution>0.01</resolution>
-                    </range>
-                    <noise>
-                        <type>gaussian</type>
-                        <mean>0.0</mean>
-                        <stddev>0.01</stddev>
-                    </noise>
-                </lidar>
-            </sensor>
-        </gazebo>
+        <xacro:lidar_3d_plugin link_reference="${name}_link" topic="/scan"/>
     </xacro:macro>
 </robot>

File: urdf/sensors/sensor_rplidar_a1.xacro (robot description, xacro)
@@ -1,4 +1,6 @@
 <?xml version="1.0"?>
 <robot xmlns:xacro="http://ros.org/wiki/xacro">
+    <!-- Include -->
+    <xacro:include filename="$(find msd700_robot_description)/urdf/gazebo/sensor_3d_lidar_gazebo.xacro"/>
     <!-- From RPLidar A1 spec -->
     <!-- https://www.slamtec.com/en/Lidar/A1 -->
@@ -44,34 +46,5 @@
             </inertial>
         </link>
-        <gazebo reference="${name}_link">
-            <sensor name="${name}_sensor" type="gpu_ray">
-                <pose>0 0 0 0 0 0</pose>
-                <topic>/scan</topic>
-                <gz_frame_id>${name}_link</gz_frame_id>
-                <update_rate>10</update_rate>
-                <always_on>true</always_on>
-                <visualize>true</visualize>
-                <ray>
-                    <scan>
-                        <horizontal>
-                            <samples>360</samples>
-                            <resolution>1</resolution>
-                            <min_angle>-3.14159</min_angle>
-                            <max_angle>3.14159</max_angle>
-                        </horizontal>
-                    </scan>
-                    <range>
-                        <min>0.15</min>
-                        <max>12.0</max>
-                        <resolution>0.01</resolution>
-                    </range>
-                    <noise>
-                        <type>gaussian</type>
-                        <mean>0.0</mean>
-                        <stddev>0.01</stddev>
-                    </noise>
-                </ray>
-            </sensor>
-        </gazebo>
+        <xacro:lidar_2d_plugin link_reference="${name}_link" topic="/scan"/>
     </xacro:macro>
 </robot>
