Commit message: fix : file path fix

File: ROS2/urdf/attachment/msd700_blade.xacro (robot description, xacro)
@@ -24,5 +24,5 @@
                 <origin xyz="0 0 0" rpy="${pi/2} 0 ${pi/2}"/>
                 <geometry>
-                    <mesh filename="package://msd700_robot_description/meshes/blade_base.dae"
+                    <mesh filename="package://msd700_robot_description/ROS2/meshes/blade_base.dae"
                         scale="1 1 1"/>
                 </geometry>
@@ -57,5 +57,5 @@
                 <origin xyz="-0.315 0 0" rpy="${pi/2} 0 ${pi/2}"/>
                 <geometry>
-                    <mesh filename="package://msd700_robot_description/meshes/blade.dae"
+                    <mesh filename="package://msd700_robot_description/ROS2/meshes/blade.dae"
                         scale="1 1 1"/>
                 </geometry>
@@ -67,5 +67,5 @@
                 <origin xyz="-0.315 0 0" rpy="${pi/2} 0 ${pi/2}"/>
                 <geometry>
-                    <mesh filename="package://msd700_robot_description/meshes/blade.dae"
+                    <mesh filename="package://msd700_robot_description/ROS2/meshes/blade.dae"
                         scale="1 1 1"/>
                 </geometry>

File: ROS2/urdf/commons/msd700_base.xacro (robot description, xacro)
@@ -22,5 +22,5 @@
                 <origin xyz="0 0 0" rpy="0 0 -${pi/2}"/>
                 <geometry>
-                    <mesh filename="package://msd700_robot_description/meshes/body_track.dae"
+                    <mesh filename="package://msd700_robot_description/ROS2/meshes/body_track.dae"
                         scale="1 1 1"/>
                 </geometry>

File: ROS2/urdf/commons/msd700_base_only.xacro (robot description, xacro)
@@ -22,5 +22,5 @@
                 <origin xyz="0 0 0" rpy="0 0 ${pi/2}"/>
                 <geometry>
-                    <mesh filename="package://msd700_robot_description/meshes/base_only.dae"
+                    <mesh filename="package://msd700_robot_description/ROS2/meshes/base_only.dae"
                         scale="1 1 1"/>
                 </geometry>

File: ROS2/urdf/commons/msd700_track.xacro (robot description, xacro)
@@ -22,5 +22,5 @@
                 <origin xyz="0 0 0" rpy="0 0 ${pi}"/>
                 <geometry>
-                    <mesh filename="package://msd700_robot_description/meshes/left_track.dae"
+                    <mesh filename="package://msd700_robot_description/ROS2/meshes/left_track.dae"
                         scale="1 1 1"/>
                 </geometry>

File: ROS2/urdf/commons/msd700_wheel.xacro (robot description, xacro)
@@ -21,5 +21,5 @@
                 <origin xyz="${(wheel_diameter/2)-0.025} ${-(wheel_length/2)+0.01} ${-((wheel_diameter/2))+0.025}" rpy="0 0 ${pi/2}"/>
                 <geometry>
-                    <mesh filename="package://msd700_robot_description/meshes/wheel.stl"
+                    <mesh filename="package://msd700_robot_description/ROS2/meshes/wheel.stl"
                             scale="0.001 0.001 0.001"/>
                 </geometry>

File: ROS2/urdf/msd700_blade_description.urdf.xacro (robot description, xacro)
@@ -2,13 +2,13 @@
 <robot name="msd700_blade" xmlns:xacro="http://ros.org/wiki/xacro">
 <!-- ================= INCLUDE ================= -->
-    <xacro:include filename="$(find msd700_robot_description)/ROS1/urdf/commons/msd700_wheel.xacro"/>
-    <xacro:include filename="$(find msd700_robot_description)/ROS1/urdf/commons/msd700_base_only.xacro"/>
-    <xacro:include filename="$(find msd700_robot_description)/ROS1/urdf/commons/msd700_track.xacro"/>
-    <xacro:include filename="$(find msd700_robot_description)/ROS1/urdf/attachment/msd700_blade.xacro"/>
-    <xacro:include filename="$(find msd700_robot_description)/ROS1/urdf/sensors/sensor_livox_360.xacro"/>
-    <xacro:include filename="$(find msd700_robot_description)/ROS1/urdf/gazebo/base_control_gazebo.xacro"/>
-    <xacro:include filename="$(find msd700_robot_description)/ROS1/urdf/gazebo/joint_state_gazebo.xacro"/>
-    <xacro:include filename="$(find msd700_robot_description)/ROS1/urdf/gazebo/sensor_2d_lidar_gazebo.xacro"/>
-    <xacro:include filename="$(find msd700_robot_description)/ROS1/urdf/gazebo/sensor_imu_gazebo.xacro"/>
+    <xacro:include filename="$(find msd700_robot_description)/ROS2/urdf/commons/msd700_wheel.xacro"/>
+    <xacro:include filename="$(find msd700_robot_description)/ROS2/urdf/commons/msd700_base_only.xacro"/>
+    <xacro:include filename="$(find msd700_robot_description)/ROS2/urdf/commons/msd700_track.xacro"/>
+    <xacro:include filename="$(find msd700_robot_description)/ROS2/urdf/attachment/msd700_blade.xacro"/>
+    <xacro:include filename="$(find msd700_robot_description)/ROS2/urdf/sensors/sensor_livox_360.xacro"/>
+    <xacro:include filename="$(find msd700_robot_description)/ROS2/urdf/gazebo/base_control_gazebo.xacro"/>
+    <xacro:include filename="$(find msd700_robot_description)/ROS2/urdf/gazebo/joint_state_gazebo.xacro"/>
+    <xacro:include filename="$(find msd700_robot_description)/ROS2/urdf/gazebo/sensor_2d_lidar_gazebo.xacro"/>
+    <xacro:include filename="$(find msd700_robot_description)/ROS2/urdf/gazebo/sensor_imu_gazebo.xacro"/>
     <xacro:property name="box_weight"       value="0.85" />
     <xacro:property name="box_width"        value="0.15" />

File: ROS2/urdf/sensors/sensor_livox_360.xacro (robot description, xacro)
@@ -22,5 +22,5 @@
                 <origin xyz="0 0 0" rpy="0 0 -${pi/2}"/>
                 <geometry>
-                    <mesh filename="package://msd700_robot_description/meshes/livox_360.dae"
+                    <mesh filename="package://msd700_robot_description/ROS2/meshes/livox_360.dae"
                         scale="1 1 1"/>
                 </geometry>
