Commit message: msd700_dump description_v1

File: src/msd700_dump_V2/urdf/model_4/attachment/msd700_dump.xacro (robot description, xacro)
@@ -2,5 +2,5 @@
 <robot xmlns:xacro="http://ros.org/wiki/xacro">
     <!-- Dimensions measured from the solid works-->
-    <xacro:property name="dump_weight"  value="50" />   <!-- from the mass properties in SW -->
+    <xacro:property name="dump_weight"  value="53.5" />
     <xacro:property name="dump_length"  value="0.805" />
     <xacro:property name="dump_width"   value="0.693" />
@@ -35,11 +35,11 @@
             </collision>
             <inertial>
-                <origin xyz="0 0 ${dump_height/2}" rpy="0 0 0"/>
+                <origin xyz="-0.0178 0.0052 0.1712" rpy="0 0 0"/>
                 <mass value="${dump_weight}"/>
                 <!-- the inertial matrix approximated as a box -->
                 <inertia
-                    ixx="${(dump_weight/12)*(dump_width*dump_width + dump_height*dump_height)}"   ixy="0.0" ixz="0.0"
-                    iyy="${(dump_weight/12)*(dump_length*dump_length + dump_height*dump_height)}" iyz="0.0"
-                    izz="${(dump_weight/12)*(dump_length*dump_length + dump_width*dump_width)}"/>
+                    ixx="2.9947" ixy="-0.0415" ixz="0.1853"
+                    iyy="4.1458" iyz="-0.0197"
+                    izz="5.6868"/>
             </inertial>
         </link>

File: src/msd700_dump_V2/urdf/model_4/common/msd700_base_stl.xacro (robot description, xacro)
@@ -2,5 +2,5 @@
 <robot xmlns:xacro="http://ros.org/wiki/xacro">
     <!-- From MCLA015B spec -->
-    <xacro:property name="base_weight"  value="121.9" />
+    <xacro:property name="base_weight"  value="144.1" />
     <xacro:property name="base_width"  value="0.47" />
     <xacro:property name="base_length"   value="0.866" />
@@ -48,11 +48,11 @@
             <inertial>
                 <mass value="${base_weight}"/>
-                <origin xyz="0 0 0.1" rpy="0 0 0"/>
+                <origin xyz="0.0901 -0.0009 0.1122" rpy="0 0 0"/>
                 <!-- the inertial matrix approximated as a box -->
                 <!-- https://en.wikipedia.org/wiki/List_of_moments_of_inertia -->
                 <inertia
-                    ixx="${(base_weight/12)*(base_width*base_width + base_height*base_height)}"   ixy="0.0" ixz="0.0"
-                    iyy="${(base_weight/12)*(base_length*base_length + base_height*base_height)}" iyz="0.0"
-                    izz="${(base_weight/12)*(base_length*base_length + base_width*base_width)}"/>
+                    ixx="4.5435" ixy="-0.0412" ixz="-0.3107"
+                    iyy="6.4175" iyz="0.0124"
+                    izz="9.0860"/>
             </inertial>
         </link>

File: src/msd700_dump_V2/urdf/model_4/common/msd700_wheel.xacro (robot description, xacro)
@@ -1,5 +1,5 @@
 <?xml version="1.0"?>
 <robot xmlns:xacro="http://ros.org/wiki/xacro">
-    <xacro:property name="wheel_weight"  value="2" />
+    <xacro:property name="wheel_weight"  value="3.5" />
     <xacro:property name="wheel_diameter"  value="0.271" />
     <xacro:property name="wheel_length"  value="0.100" />
@@ -38,7 +38,7 @@
                 <mass value="${wheel_weight}"/>
                 <inertia
-                    ixx="${1/12*wheel_weight*(3*(wheel_diameter/2)*(wheel_diameter/2) + wheel_length * wheel_length)}"
-                    iyy="${1/12*wheel_weight*(3*(wheel_diameter/2)*(wheel_diameter/2) + wheel_length * wheel_length)}"
-                    izz="${wheel_weight/2*(wheel_diameter/2)*(wheel_diameter/2)}"
+                    ixx="0.0153"
+                    iyy="0.0153"
+                    izz="0.0280"
                     ixy="0" ixz="0" iyz="0"/>
             </inertial>

File: src/msd700_dump_V2/urdf/model_4/sensors/sensor_airy.xacro (robot description, xacro)
@@ -1,13 +1,9 @@
 <?xml version="1.0"?>
 <robot xmlns:xacro="http://ros.org/wiki/xacro">
-    <!-- RoboSense Airy lidar (MCLA022A_Airy_LIDAR.STL, includes the mount plate and bracket) -->
     <!-- Head dimensions measured from the STL -->
-    <xacro:property name="airy_weight"  value="0.35" />   <!-- TODO: real mass -->
+    <xacro:property name="airy_weight"  value="0.35" />
     <xacro:property name="airy_length"  value="0.106" />
     <xacro:property name="airy_width"   value="0.100" />
     <xacro:property name="airy_height"  value="0.094" />
-    <!-- The link origin is the centre of the lidar head.
-         The STL origin is not at the head, so the visual is shifted back to it.
-         Use the link name as the driver frame_id (lidar_airy.yaml: ros_frame_id). -->
     <xacro:macro name="airy" params="
         name
@@ -40,9 +36,8 @@
                 <origin xyz="0 0 0" rpy="0 0 0"/>
                 <mass value="${airy_weight}"/>
-                <!-- the inertial matrix approximated as a box -->
                 <inertia
-                    ixx="${(airy_weight/12)*(airy_width*airy_width + airy_height*airy_height)}"   ixy="0.0" ixz="0.0"
-                    iyy="${(airy_weight/12)*(airy_length*airy_length + airy_height*airy_height)}" iyz="0.0"
-                    izz="${(airy_weight/12)*(airy_length*airy_length + airy_width*airy_width)}"/>
+                    ixx="${(airy_weight/12)*(3*0.0375*0.0375 + 0.070*0.070)}"   ixy="0.0" ixz="0.0"
+                    iyy="${(airy_weight/12)*(3*0.0375*0.0375 + 0.070*0.070)}" iyz="0.0"
+                    izz="${(airy_weight/2)*(0.0375*0.0375)}"/>
             </inertial>
         </link>

File: src/msd700_dump_V2/urdf/model_4/sensors/sensor_e1r.xacro (robot description, xacro)
@@ -1,14 +1,9 @@
 <?xml version="1.0"?>
 <robot xmlns:xacro="http://ros.org/wiki/xacro">
-    <!-- RoboSense E1R lidar (MCLA022A_E1R_LIDAR.STL, includes the mount bracket) -->
     <!-- Head dimensions measured from the STL -->
-    <xacro:property name="e1r_weight"  value="0.33" />   <!-- TODO: real mass -->
+    <xacro:property name="e1r_weight"  value="0.33" />
     <xacro:property name="e1r_length"  value="0.089" />
     <xacro:property name="e1r_width"   value="0.182" />
     <xacro:property name="e1r_height"  value="0.125" />
-    <!-- The link origin is the centre of the lidar head, X = viewing direction.
-         The STL was exported in the dump assembly frame (not its own origin),
-         so the visual is shifted back from the head centre to the assembly origin.
-         Use the link name as the driver frame_id (lidar_e1r.yaml: ros_frame_id). -->
     <xacro:macro name="e1r" params="
         name
@@ -43,7 +38,7 @@
                 <!-- the inertial matrix approximated as a box -->
                 <inertia
-                    ixx="${(e1r_weight/12)*(e1r_width*e1r_width + e1r_height*e1r_height)}"   ixy="0.0" ixz="0.0"
-                    iyy="${(e1r_weight/12)*(e1r_length*e1r_length + e1r_height*e1r_height)}" iyz="0.0"
-                    izz="${(e1r_weight/12)*(e1r_length*e1r_length + e1r_width*e1r_width)}"/>
+                    ixx="${(e1r_weight/12)*(0.095*0.095 + 0.043*0.043)}"   ixy="0.0" ixz="0.0"
+                    iyy="${(e1r_weight/12)*(0.0695*0.0695 + 0.043*0.043)}" iyz="0.0"
+                    izz="${(e1r_weight/12)*(0.0695*0.0695 + 0.095*0.095)}"/>
             </inertial>
         </link>
